File: RPi-Ham/RPi-Ham.kicad_pcb (KiCad board)
At the start: 2 copper layers, 65 x 56.5 mm, 44 parts, among them J1 Conn_02x03_Counter_Clockwise, J10 MountingHole_2.7mm_M2.5_Pad_V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, J11 MountingHole_2.7mm_M2.5_Pad_V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, J12 MountingHole_2.7mm_M2.5_Pad_V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, J13 MountingHole_2.7mm_M2.5_Pad_V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, J2 RJ45, J3 Conn_02x03_Counter_Clockwise, J4 RJ45, J5 RJ45, J6 Conn_02x08_Counter_Clockwise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

Commit message: Added mount for pi zero
Parts:
- added J13: MountingHole_2.7mm_M2.5_Pad_Via, MountingHole:MountingHole_2.7mm_M2.5_Pad_Via, F.Cu at (51.0, 55.5)
Changed lines of the file:
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@@
     (tracks 574)
     (zones 0)
-    (modules 44)
+    (modules 45)
     (nets 95)
   )
@@
     (visible_elements FFFFE7FF)
     (pcbplotparams
-      (layerselection 0x010fc_ffffffff)
+      (layerselection 0x010f0_ffffffff)
       (usegerberextensions false)
       (usegerberattributes false)
@@
       (outputformat 1)
       (mirror false)
-      (drillshape 1)
+      (drillshape 0)
       (scaleselection 1)
       (outputdirectory ""))
@@
     (add_net VCC)
     (add_net VDD)
+  )
+  (module MountingHole:MountingHole_2.7mm_M2.5_Pad_Via (layer F.Cu)
+    (at 51 55.5)
+    (descr "Mounting Hole 2.7mm")
+    (tags "mounting hole 2.7mm")
+    (attr virtual)
+    (fp_text reference J13 (at 0 0) (layer F.SilkS)
+      (effects (font (size 1 1) (thickness 0.15)))
+    )
+    (fp_text value MountingHole_2.7mm_M2.5_Pad_Via (at 0 3.7) (layer F.Fab)
+      (effects (font (size 1 1) (thickness 0.15)))
+    )
+    (fp_text user %R (at 0.3 0) (layer F.Fab)
+      (effects (font (size 1 1) (thickness 0.15)))
+    )
+    (fp_circle (center 0 0) (end 2.7 0) (layer Cmts.User) (width 0.15))
+    (fp_circle (center 0 0) (end 2.95 0) (layer F.CrtYd) (width 0.05))
+    (pad 1 thru_hole circle (at 0 0) (size 5.4 5.4) (drill 2.7) (layers *.Cu *.Mask))
+    (pad 1 thru_hole circle (at 2.025 0) (size 0.8 0.8) (drill 0.5) (layers *.Cu *.Mask))
+    (pad 1 thru_hole circle (at 1.431891 1.431891) (size 0.8 0.8) (drill 0.5) (layers *.Cu *.Mask))
+    (pad 1 thru_hole circle (at 0 2.025) (size 0.8 0.8) (drill 0.5) (layers *.Cu *.Mask))
+    (pad 1 thru_hole circle (at -1.431891 1.431891) (size 0.8 0.8) (drill 0.5) (layers *.Cu *.Mask))
+    (pad 1 thru_hole circle (at -2.025 0) (size 0.8 0.8) (drill 0.5) (layers *.Cu *.Mask))
+    (pad 1 thru_hole circle (at -1.431891 -1.431891) (size 0.8 0.8) (drill 0.5) (layers *.Cu *.Mask))
+    (pad 1 thru_hole circle (at 0 -2.025) (size 0.8 0.8) (drill 0.5) (layers *.Cu *.Mask))
+    (pad 1 thru_hole circle (at 1.431891 -1.431891) (size 0.8 0.8) (drill 0.5) (layers *.Cu *.Mask))
   )
   (module RPi-Ham:logo (layer B.Cu)
@@
     )
   )
-  (gr_text "HAM Radio Interface v1.0" (at 54.5 56.75 90) (layer B.SilkS)
+  (gr_text "HAM Radio Interface v1.0" (at 55.25 56.75 90) (layer B.SilkS)
     (effects (font (size 1.5 1.5) (thickness 0.3)) (justify mirror))
   )
@@
     (effects (font (size 1.5 1.5) (thickness 0.3)))
   )
-  (gr_text "Audio 1" (at 54.75 60) (layer F.SilkS)
+  (gr_text "Audio 1" (at 58.25 60.25) (layer F.SilkS)
     (effects (font (size 1.5 1.5) (thickness 0.3)))
   )
-  (gr_text "Audio 0" (at 54.75 54) (layer F.SilkS)
+  (gr_text "Audio 0" (at 58.25 54) (layer F.SilkS)
     (effects (font (size 1.5 1.5) (thickness 0.3)))
   )
